Commit message: Correct urdf orientation in RVIZ and comment out  envelope reference

File: src/meca500_scene_description/urdf/scene.urdf.xacro (robot description, xacro)
@@ -5,6 +5,12 @@
   <!-- Shared reference frame = your Onshape assembly origin -->
   <link name="world"/>
+  <link name="scene_frame"/>
+  <joint name="world_to_scene" type="fixed">
+    <parent link="world"/>
+    <child link="scene_frame"/>
+    <origin xyz="0 0 0" rpy="-1.5708 0 0"/>
+  </joint>
   <!-- Robot, offset from world by the measured mount position -->
-  <xacro:meca500 parent="world">
+  <xacro:meca500 parent="scene_frame">
     <origin xyz="-0.15 -0.0127 0" rpy="1.5708 0 0"/>
   </xacro:meca500>
@@ -82,6 +88,6 @@
     </visual>
   </link>
-  <joint name="world_to_breadboard" type="fixed">
-    <parent link="world"/>
+  <joint name="scene_to_breadboard" type="fixed">
+    <parent link="scene_frame"/>
     <child link="breadboard"/>
     <origin xyz="0 0 0" rpy="0 0 0"/>
@@ -100,9 +106,9 @@
   </link>
   <joint name="world_to_phantom" type="fixed">
-    <parent link="world"/>
+    <parent link="scene_frame"/>
     <child link="phantom"/>
     <origin xyz="0.164 -0.0427 0 " rpy="1.5708 3.14159 3.14159"/>
   </joint>
-  <!-- Reach envelope reference (Mecademic-published workspace shape), translucent -->
+  <!-- Reach envelope reference (Mecademic-published workspace shape), translucent
   <link name="workspace_envelope">
     <visual>
@@ -119,5 +125,6 @@
     <parent link="base_link"/>
     <child link="workspace_envelope"/>
-    <origin xyz="0 0 0" rpy="-1.5708 -3.14159 -1.5708"/>
+    <origin xyz="0 0 0" rpy="1.5708 0 3.14159"/>
   </joint>
+</robot> -->
 </robot>

Commit message: Fix MoveIt OMPL planning pipeline for ROS 2 Lyrical

File: src/meca500_scene_description/urdf/scene.urdf.xacro (robot description, xacro)
@@ -104,4 +104,10 @@
       </material>
     </visual>
+    <collision>
+      <origin xyz="0 0 0" rpy="0 0 0"/>
+      <geometry>
+        <mesh filename="package://meca500_scene_description/meshes/phantom.stl" scale="0.001 0.001 0.001"/>
+      </geometry>
+    </collision>
   </link>
   <joint name="world_to_phantom" type="fixed">

Commit message: Collision logic fixed

File: src/meca500_scene_description/urdf/scene.urdf.xacro (robot description, xacro)
@@ -26,4 +26,10 @@
       </material>
     </visual>
+    <collision>
+      <origin xyz="0 0 0" rpy="0 0 0"/>
+      <geometry>
+        <mesh filename="package://meca500_scene_description/meshes/bottom.stl" scale="0.001 0.001 0.001"/>
+      </geometry>
+    </collision>
   </link>
   <joint name="link6_to_camera_adapter_bottom" type="fixed">
@@ -43,4 +49,10 @@
       </material>
     </visual>
+    <collision>
+      <origin xyz="0 0 0" rpy="0 0 0"/>
+      <geometry>
+        <mesh filename="package://meca500_scene_description/meshes/top.stl" scale="0.001 0.001 0.001"/>
+      </geometry>
+    </collision>
   </link>
   <joint name="adapter_bottom_to_top" type="fixed">
@@ -60,4 +72,10 @@
       </material>
     </visual>
+    <collision>
+      <origin xyz="0 0 0" rpy="1.5708 0 0"/>
+      <geometry>
+        <mesh filename="package://meca500_scene_description/meshes/camera.stl" scale="0.001 0.001 0.001"/>
+      </geometry>
+    </collision>
   </link>
   <joint name="adapter_to_camera" type="fixed">
@@ -87,4 +105,10 @@
       </material>
     </visual>
+    <collision>
+      <origin xyz="0 0 0" rpy="3.14159 0 0"/>
+      <geometry>
+        <mesh filename="package://meca500_scene_description/meshes/breadboard.stl" scale="0.001 0.001 0.001"/>
+      </geometry>
+    </collision>
   </link>
   <joint name="scene_to_breadboard" type="fixed">

Commit message: Enable MoveIt simulated execution with mock hardware

File: src/meca500_scene_description/urdf/scene.urdf.xacro (robot description, xacro)
@@ -140,4 +140,25 @@
     <origin xyz="0.164 -0.0427 0 " rpy="1.5708 3.14159 3.14159"/>
   </joint>
+  <!-- Laptop simulation: joint commands become simulated positions -->
+  <xacro:macro name="mock_joint" params="name">
+    <joint name="${name}">
+      <command_interface name="position"/>
+      <state_interface name="position">
+        <param name="initial_value">0.0</param>
+      </state_interface>
+      <state_interface name="velocity"/>
+    </joint>
+  </xacro:macro>
+  <ros2_control name="Meca500MockSystem" type="system">
+    <hardware>
+      <plugin>mock_components/GenericSystem</plugin>
+    </hardware>
+    <xacro:mock_joint name="meca_axis_1"/>
+    <xacro:mock_joint name="meca_axis_2"/>
+    <xacro:mock_joint name="meca_axis_3"/>
+    <xacro:mock_joint name="meca_axis_4"/>
+    <xacro:mock_joint name="meca_axis_5"/>
+    <xacro:mock_joint name="meca_axis_6"/>
+  </ros2_control>
   <!-- Reach envelope reference (Mecademic-published workspace shape), translucent
   <link name="workspace_envelope">
